Commit message: set cube to cube geometry

File: examples/05-kuka_pick_and_place/resources/cube.urdf (robot description, URDF)
Before this commit: robot cube, 7 links, 6 joints
Links:
- link object: geometry collision box size=0.1 0.1 0.1; visual box size=0.1 0.1 0.1

File: examples/05-kuka_pick_and_place/resources/kuka_iiwa.urdf (robot description, URDF)
Before this commit: robot kuka_iiwa, 10 links, 9 joints
Links:
- link link6: geometry collision box size=0.08 0.08 0.08; visual box size=0.1 0.1 0.1
