Commit message: bugfixes and examples cleanup

File: examples/10-3d_orientation_controller/panda_arm.urdf (robot description, URDF)
Before this commit: robot panda, 9 links, 8 joints
Links:
- link end-effector: geometry collision sphere radius=0.04; visual sphere radius=0.04
Joints:
- joint joint_ee: origin xyz=0 0 0.14 rpy=0 0 0 -> xyz=0 0 0.15 rpy=0 0 0
