Commit message: updates for new rbdl + eigen compatilility

File: examples/21-singularity/panda_arm.urdf (robot description, URDF)
Before this commit: robot panda, 9 links, 8 joints
Joints:
- joint joint4: limit lower=-3.0718 upper=-0.5 effort=87 velocity=2.1750 -> lower=-3.0718 upper=-0.0698 effort=87 velocity=2.1750
