Commit message: cleaned up examples to make them use global robot models defined in sai2Model

File: examples/06-partial_joint_task/panda_arm_sliding_base.urdf (robot description, URDF)
Before this commit: robot panda, 10 links, 9 joints
Links:
- link link0: geometry visual mesh filename=${SAI2_MODEL_URDF_FOLDER}/panda/meshes/visual/link0.obj
- link link1: geometry visual mesh filename=${SAI2_MODEL_URDF_FOLDER}/panda/meshes/visual/link1.obj
- link link2: geometry visual mesh filename=${SAI2_MODEL_URDF_FOLDER}/panda/meshes/visual/link2.obj
- link link3: geometry visual mesh filename=${SAI2_MODEL_URDF_FOLDER}/panda/meshes/visual/link3.obj
- link link4: geometry visual mesh filename=${SAI2_MODEL_URDF_FOLDER}/panda/meshes/visual/link4.obj
- link link5: geometry visual mesh filename=${SAI2_MODEL_URDF_FOLDER}/panda/meshes/visual/link5.obj
- link link6: geometry visual mesh filename=${SAI2_MODEL_URDF_FOLDER}/panda/meshes/visual/link6.obj
- link link7: geometry visual mesh filename=${SAI2_MODEL_URDF_FOLDER}/panda/meshes/visual/link7.obj

File: examples/15-haptic_control_impedance_type/panda_arm.urdf (robot description, URDF)
Before this commit: robot panda, 9 links, 8 joints
Links:
- link link0: geometry visual mesh filename=${SAI2_MODEL_URDF_FOLDER}/panda/meshes/visual/link0.obj
- link link1: geometry visual mesh filename=${SAI2_MODEL_URDF_FOLDER}/panda/meshes/visual/link1.obj
- link link2: geometry visual mesh filename=${SAI2_MODEL_URDF_FOLDER}/panda/meshes/visual/link2.obj
- link link3: geometry visual mesh filename=${SAI2_MODEL_URDF_FOLDER}/panda/meshes/visual/link3.obj
- link link4: geometry visual mesh filename=${SAI2_MODEL_URDF_FOLDER}/panda/meshes/visual/link4.obj
- link link5: geometry visual mesh filename=${SAI2_MODEL_URDF_FOLDER}/panda/meshes/visual/link5.obj
- link link6: geometry visual mesh filename=${SAI2_MODEL_URDF_FOLDER}/panda/meshes/visual/link6.obj
- link link7: geometry visual mesh filename=${SAI2_MODEL_URDF_FOLDER}/panda/meshes/visual/link7.obj

File: examples/17-bilateral_teleop_with_POPC/panda_arm.urdf (robot description, URDF)
Before this commit: robot panda, 9 links, 8 joints
Links:
- link link0: geometry visual mesh filename=${SAI2_MODEL_URDF_FOLDER}/panda/meshes/visual/link0.obj
- link link1: geometry visual mesh filename=${SAI2_MODEL_URDF_FOLDER}/panda/meshes/visual/link1.obj
- link link2: geometry visual mesh filename=${SAI2_MODEL_URDF_FOLDER}/panda/meshes/visual/link2.obj
- link link3: geometry visual mesh filename=${SAI2_MODEL_URDF_FOLDER}/panda/meshes/visual/link3.obj
- link link4: geometry visual mesh filename=${SAI2_MODEL_URDF_FOLDER}/panda/meshes/visual/link4.obj
- link link5: geometry visual mesh filename=${SAI2_MODEL_URDF_FOLDER}/panda/meshes/visual/link5.obj
- link link6: geometry visual mesh filename=${SAI2_MODEL_URDF_FOLDER}/panda/meshes/visual/link6.obj
- link link7: geometry visual mesh filename=${SAI2_MODEL_URDF_FOLDER}/panda/meshes/visual/link7.obj

Commit message: rename sai2 to sai

File: examples/06-partial_joint_task/panda_arm_sliding_base.urdf (robot description, URDF)
Before this commit: robot panda, 10 links, 9 joints
Links:
- link link0: geometry visual mesh filename=${SAI_MODEL_URDF_FOLDER}/panda/meshes/visual/link0.obj
- link link1: geometry visual mesh filename=${SAI_MODEL_URDF_FOLDER}/panda/meshes/visual/link1.obj
- link link2: geometry visual mesh filename=${SAI_MODEL_URDF_FOLDER}/panda/meshes/visual/link2.obj
- link link3: geometry visual mesh filename=${SAI_MODEL_URDF_FOLDER}/panda/meshes/visual/link3.obj
- link link4: geometry visual mesh filename=${SAI_MODEL_URDF_FOLDER}/panda/meshes/visual/link4.obj
- link link5: geometry visual mesh filename=${SAI_MODEL_URDF_FOLDER}/panda/meshes/visual/link5.obj
- link link6: geometry visual mesh filename=${SAI_MODEL_URDF_FOLDER}/panda/meshes/visual/link6.obj
- link link7: geometry visual mesh filename=${SAI_MODEL_URDF_FOLDER}/panda/meshes/visual/link7.obj

File: examples/15-haptic_control_impedance_type/panda_arm.urdf (robot description, URDF)
Before this commit: robot panda, 9 links, 8 joints
Links:
- link link0: geometry visual mesh filename=${SAI_MODEL_URDF_FOLDER}/panda/meshes/visual/link0.obj
- link link1: geometry visual mesh filename=${SAI_MODEL_URDF_FOLDER}/panda/meshes/visual/link1.obj
- link link2: geometry visual mesh filename=${SAI_MODEL_URDF_FOLDER}/panda/meshes/visual/link2.obj
- link link3: geometry visual mesh filename=${SAI_MODEL_URDF_FOLDER}/panda/meshes/visual/link3.obj
- link link4: geometry visual mesh filename=${SAI_MODEL_URDF_FOLDER}/panda/meshes/visual/link4.obj
- link link5: geometry visual mesh filename=${SAI_MODEL_URDF_FOLDER}/panda/meshes/visual/link5.obj
- link link6: geometry visual mesh filename=${SAI_MODEL_URDF_FOLDER}/panda/meshes/visual/link6.obj
- link link7: geometry visual mesh filename=${SAI_MODEL_URDF_FOLDER}/panda/meshes/visual/link7.obj

File: examples/17-bilateral_teleop_with_POPC/panda_arm.urdf (robot description, URDF)
Before this commit: robot panda, 9 links, 8 joints
Links:
- link link0: geometry visual mesh filename=${SAI_MODEL_URDF_FOLDER}/panda/meshes/visual/link0.obj
- link link1: geometry visual mesh filename=${SAI_MODEL_URDF_FOLDER}/panda/meshes/visual/link1.obj
- link link2: geometry visual mesh filename=${SAI_MODEL_URDF_FOLDER}/panda/meshes/visual/link2.obj
- link link3: geometry visual mesh filename=${SAI_MODEL_URDF_FOLDER}/panda/meshes/visual/link3.obj
- link link4: geometry visual mesh filename=${SAI_MODEL_URDF_FOLDER}/panda/meshes/visual/link4.obj
- link link5: geometry visual mesh filename=${SAI_MODEL_URDF_FOLDER}/panda/meshes/visual/link5.obj
- link link6: geometry visual mesh filename=${SAI_MODEL_URDF_FOLDER}/panda/meshes/visual/link6.obj
- link link7: geometry visual mesh filename=${SAI_MODEL_URDF_FOLDER}/panda/meshes/visual/link7.obj
